File: kicad/LF_phase_detector.kicad_pcb (KiCad board)
At the start: 2 copper layers, 108 x 99.8 mm, 233 parts, among them M1 NUCLEO-H743ZI, P1 MSTBA 2,5/ 2-G-5,08 - 1757242, T1 AO4485, U1 HMC984LP4E, U10 TMUX1204DGSR, U11 TMUX1204DGSR, U12 TMUX1204DGSR, U13 TMUX1204DGSR, U14 OPA2325, U15 ADA4807-2ARM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

Commit message: some initial commits
Other:
- net class 24V removed
- net class Default removed
- net class motor removed
- net class motorii removed
- net class zasilanie 5v removed
